File: alps64.kicad_pcb (KiCad board)
At the start: 2 copper layers, 152.1 x 100.3 mm, 27 parts, among them J2 USB_C_Receptacle, K18 keyboard_parts:KEYSW, K19 keyboard_parts:KEYSW, K28 keyboard_parts:KEYSW, K29 keyboard_parts:KEYSW, K8 keyboard_parts:KEYSW, K9 keyboard_parts:KEYSW, SW100 SW_PUSH, U1 32U2, Y1 Crystal_GND24

Commit message: Use through hall led footprint
Parts:
- LED1: footprint LED_SMD:LED_0805_2012Metric_Pad1.15x1.40mm_HandSolder -> LED_THT:LED_D3.0mm
Changed lines of the file:
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@@
     )
   )
-  (footprint "LED_SMD:LED_0805_2012Metric_Pad1.15x1.40mm_HandSolder" (layer "F.Cu")
+  (footprint "LED_THT:LED_D3.0mm" (layer "F.Cu")
     (at 153.65 124.85)
-    (descr "LED SMD 0805 (2012 Metric), square (rectangular) end terminal, IPC_7351 nominal, (Body size source: https://docs.google.com/spreadsheets/d/1BsfQQcO9C6DZCsRaXUlFlo91Tg2WpOkGARC1WS5S8t0/edit?usp=sharing), generated with kicad-footprint-generator")
-    (tags "LED handsolder")
+    (descr "LED, diameter 3.0mm, 2 pins")
+    (tags "LED diameter 3.0mm 2 pins")
     (property "Sheetfile" "alps64.kicad_sch")
     (property "Sheetname" "")
-    (attr smd)
-    (fp_text reference "LED1" (at 0 -1.65) (layer "F.SilkS")
+    (attr through_hole)
+    (fp_text reference "LED1" (at 1.27 -2.96) (layer "F.SilkS")
         (effects (font (size 1 1) (thickness 0.15)))
     )
-    (fp_text value "LED" (at 0 1.65) (layer "F.Fab")
+    (fp_text value "LED" (at 1.27 2.96) (layer "F.Fab")
         (effects (font (size 1 1) (thickness 0.15)))
     )
-    (fp_text user "${REFERENCE}" (at 0 0) (layer "F.Fab")
-        (effects (font (size 0.5 0.5) (thickness 0.08)))
-    )
-    (fp_line (start -1.86 -0.96) (end -1.86 0.96)
+    (fp_line (start -0.29 -1.236) (end -0.29 -1.08)
       (stroke (width 0.12) (type solid)) (layer "F.SilkS"))
-    (fp_line (start -1.86 0.96) (end 1 0.96)
+    (fp_line (start -0.29 1.08) (end -0.29 1.236)
       (stroke (width 0.12) (type solid)) (layer "F.SilkS"))
-    (fp_line (start 1 -0.96) (end -1.86 -0.96)
+    (fp_arc (start -0.29 -1.235516) (mid 1.366487 -1.987659) (end 2.942335 -1.078608)
       (stroke (width 0.12) (type solid)) (layer "F.SilkS"))
-    (fp_line (start -1.85 -0.95) (end 1.85 -0.95)
+    (fp_arc (start 0.229039 -1.08) (mid 1.270117 -1.5) (end 2.31113 -1.079837)
+      (stroke (width 0.12) (type solid)) (layer "F.SilkS"))
+    (fp_arc (start 2.31113 1.079837) (mid 1.270117 1.5) (end 0.229039 1.08)
+      (stroke (width 0.12) (type solid)) (layer "F.SilkS"))
+    (fp_arc (start 2.942335 1.078608) (mid 1.366487 1.987659) (end -0.29 1.235516)
+      (stroke (width 0.12) (type solid)) (layer "F.SilkS"))
+    (fp_line (start -1.15 -2.25) (end -1.15 2.25)
       (stroke (width 0.05) (type solid)) (layer "F.CrtYd"))
-    (fp_line (start -1.85 0.95) (end -1.85 -0.95)
+    (fp_line (start -1.15 2.25) (end 3.7 2.25)
       (stroke (width 0.05) (type solid)) (layer "F.CrtYd"))
-    (fp_line (start 1.85 -0.95) (end 1.85 0.95)
+    (fp_line (start 3.7 -2.25) (end -1.15 -2.25)
       (stroke (width 0.05) (type solid)) (layer "F.CrtYd"))
-    (fp_line (start 1.85 0.95) (end -1.85 0.95)
+    (fp_line (start 3.7 2.25) (end 3.7 -2.25)
       (stroke (width 0.05) (type solid)) (layer "F.CrtYd"))
-    (fp_line (start -1 -0.3) (end -1 0.6)
+    (fp_line (start -0.23 -1.16619) (end -0.23 1.16619)
       (stroke (width 0.1) (type solid)) (layer "F.Fab"))
-    (fp_line (start -1 0.6) (end 1 0.6)
+    (fp_arc (start -0.23 -1.16619) (mid 3.17 0.000452) (end -0.230555 1.165476)
       (stroke (width 0.1) (type solid)) (layer "F.Fab"))
-    (fp_line (start -0.7 -0.6) (end -1 -0.3)
-      (stroke (width 0.1) (type solid)) (layer "F.Fab"))
-    (fp_line (start 1 -0.6) (end -0.7 -0.6)
-      (stroke (width 0.1) (type solid)) (layer "F.Fab"))
-    (fp_line (start 1 0.6) (end 1 -0.6)
-      (stroke (width 0.1) (type solid)) (layer "F.Fab"))
-    (pad "1" smd roundrect (at -1.025 0) (size 1.15 1.4) (layers "F.Cu" "F.Paste" "F.Mask") (roundrect_rratio 0.217391)
+    (fp_circle (center 1.27 0) (end 2.77 0)
+      (stroke (width 0.1) (type solid)) (fill none) (layer "F.Fab"))
+    (pad "1" thru_hole rect (at 0 0) (size 1.8 1.8) (drill 0.9) (layers "*.Cu" "*.Mask")
       (net 18 "Net-(LED1-K)") (pinfunction "K") (pintype "passive"))
-    (pad "2" smd roundrect (at 1.025 0) (size 1.15 1.4) (layers "F.Cu" "F.Paste" "F.Mask") (roundrect_rratio 0.217391)
+    (pad "2" thru_hole circle (at 2.54 0) (size 1.8 1.8) (drill 0.9) (layers "*.Cu" "*.Mask")
       (net 19 "Net-(LED1-A)") (pinfunction "A") (pintype "passive"))
-    (model "${KICAD6_3DMODEL_DIR}/LED_SMD.3dshapes/LED_0805_2012Metric.wrl"
+    (model "${KICAD6_3DMODEL_DIR}/LED_THT.3dshapes/LED_D3.0mm.wrl"
       (offset (xyz 0 0 0))
       (scale (xyz 1 1 1))
